File: file60B795C7.sch (KiCad schematic (older format))
At the start: 11 parts, among them J101 bass guitar input, J103 iso output, J104 XLR out

Commit message: defined mounting holes, and 1 chassis mounting hole and star ground point removed all guitar related parts to create the royermod psu on its own need to define switch to toggle 39k cathode resistor
exported gerbers for test build

still need:
front panel
bom
will define this as a release after double checking
Parts:
- V101: footprint Valve: flat pins -> Connector_PinHeader_1.27mm:PinHeader_1x07_P1.27mm_Vertical
Changed lines of the file:
@@
 F 0 "V101" H 3625 3481 50  0000 C CNN
 F 1 "S290MS001P003" H 3625 3390 50  0000 C CNN
-F 2 "Valve: flat pins" H 3150 2400 50  0001 C CNN
+F 2 "Connector_PinHeader_1.27mm:PinHeader_1x07_P1.27mm_Vertical" H 3150 2400 50  0001 C CNN
 F 3 "http://www.r-type.org/pdfs/el34.pdf" H 3650 2950 50  0001 C CNN
 	1    3650 2850
